File: IMD_Carrier/IMD_Carrier.kicad_pcb (KiCad board)
At the start: 2 copper layers, 158 x 118 mm, 34 parts, among them J1 JST-XA, J2 MicroFit+, J3 JST-XA, J4 MicroFit+, K2 Relay_SPDT_G6RN, Q1 BSS205N, Q2 BSS205N, Q6 BSS205N, U1 CD4043BE, U2 TLV1702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

Commit message: finished the routing of the PCB (to be checked)
Parts:
- removed J4: MicroFit+, Custom_MSM:Connector_MicroFit-Plus_2POS
- removed U3: 74AUC2G00, Custom_MSM:74AHC2G00DC-Q100
- added IC1: CD4012BM96, Custom_MSM:Dual NAND, Quad input, F.Cu at (132.8, 132.5)
- R3: value R -> 470
- R7: value R -> 10k
- moved J2 48.1 mm to (252.5, 71.5)
Connections:
- J2 pad 1: HV- -> HV+
- U2 pad 4: unconnected-(U2C-V--Pad4) -> GND
- U2 pad 8: unconnected-(U2C-V+-Pad8) -> +12V
Routing:
- net +12V: track 0.00 -> 378.9 mm, vias 0 -> 5

Commit message: Add files via upload
Routing:
- net IMD_Latch: track 10.4 -> 25.3 mm, vias 0 -> 1
- added copper zone on B.Cu, net (none)
- added copper zone on F.Cu, net (none)
Changed lines of the file:
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@@
 	)
 	(setup
+		(stackup
+			(layer "F.SilkS"
+				(type "Top Silk Screen")
+			)
+			(layer "F.Paste"
+				(type "Top Solder Paste")
+			)
+			(layer "F.Mask"
+				(type "Top Solder Mask")
+				(thickness 0.01)
+			)
+			(layer "F.Cu"
+				(type "copper")
+				(thickness 0.035)
+			)
+			(layer "dielectric 1"
+				(type "core")
+				(thickness 1.51)
+				(material "FR4")
+				(epsilon_r 4.5)
+				(loss_tangent 0.02)
+			)
+			(layer "B.Cu"
+				(type "copper")
+				(thickness 0.035)
+			)
+			(layer "B.Mask"
+				(type "Bottom Solder Mask")
+				(thickness 0.01)
+			)
+			(layer "B.Paste"
+				(type "Bottom Solder Paste")
+			)
+			(layer "B.SilkS"
+				(type "Bottom Silk Screen")
+			)
+			(copper_finish "None")
+			(dielectric_constraints no)
+		)
 		(pad_to_mask_clearance 0)
 		(allow_soldermask_bridges_in_footprints no)
@@
 	)
 	(segment
-		(start 148.58 35.55)
-		(end 141.45 35.55)
+		(start 148.13 36)
+		(end 148.58 35.55)
 		(width 0.2)
 		(layer "F.Cu")
@@
 	)
 	(segment
-		(start 141.45 35.55)
-		(end 139.5 37.5)
+		(start 147 36)
+		(end 148.13 36)
 		(width 0.2)
 		(layer "F.Cu")
 		(net 14)
 	)
+	(via
+		(at 147 36)
+		(size 0.6)
+		(drill 0.3)
+		(layers "F.Cu" "B.Cu")
+		(net 14)
+	)
+	(segment
+		(start 147 44.5)
+		(end 147 36)
+		(width 0.2)
+		(layer "B.Cu")
+		(net 14)
+	)
 	(segment
 		(start 131.575 134.75)
@@
 	)
 	(segment
+		(start 139.5 44.5)
+		(end 147 44.5)
+		(width 0.2)
+		(layer "B.Cu")
+		(net 14)
+	)
+	(segment
+		(start 139.4125 44.4125)
+		(end 139.5 44.5)
+		(width 0.2)
+		(layer "B.Cu")
+		(net 14)
+	)
+	(segment
+		(start 139.4125 37.5)
+		(end 139.4125 44.4125)
+		(width 0.2)
+		(layer "B.Cu")
+		(net 14)
+	)
+	(segment
 		(start 152 36.5)
 		(end 158.5 30)
@@
 		(net 39)
 	)
+	(zone
+		(net 0)
+		(net_name "")
+		(layers "F.Cu" "B.Cu")
+		(hatch edge 0.5)
+		(connect_pads
+			(clearance 0.5)
+		)
+		(min_thickness 0.25)
+		(filled_areas_thickness no)
+		(fill yes
+			(thermal_gap 0.5)
+			(thermal_bridge_width 0.5)
+			(island_removal_mode 1)
+			(island_area_min 10)
+		)
+		(polygon
+			(pts
+				(xy 252 22.5) (xy 252.5 140.5) (xy 97 139.5) (xy 100.5 22.5)
+			)
+		)
+	)
 	(embedded_fonts no)
