File: IMD_Carrier/IMD_Carrier.kicad_pcb (KiCad board)
At the start: 2 copper layers, 158 x 118 mm, 39 parts, among them IC1 CD4012BM96, J1 JST-XA, J2 MicroFit+, J3 JST-XA, J4 JST-XA, J5 JST-XA, K2 Relay_SPDT_G6RN, Q1 BSS205N, Q2 BSS205N, Q6 BSS205N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

Commit message: Add files via upload
Parts:
- removed the G*** at (244.6, 113.2)
- added U3: LM2596S, Package_TO_SOT_SMD:TO-263-5_TabPin3, F.Cu at (10.2, 5.67)
- R10: value 8.5k -> 17k
- R11: value 3.5k -> 31k
- R8: value 2.5k -> 29k
- R9: value 9.5k -> 19k
Connections:
- D4 pad 1: +12V -> +24V
- J1 pad 1: GND -> +5V
- J1 pad 2: +12V -> +24V
- J2 pad 2: HV- -> HV+
- J4 pad 1: +12V -> Net-(J4-Pin_1)
- J4 pad 4: GND -> +5V
- K2 pad 5: +12V -> +24V
- Q1 pad 2: GND -> +5V
- Q2 pad 2: GND -> +5V
- Q6 pad 2: GND -> +5V
- R1 pad 2: GND -> +5V
- R10 pad 2: GND -> +5V
- R11 pad 2: +12V -> +24V
- R13 pad 1: +12V -> +5V
- R2 pad 2: GND -> +5V
- R8 pad 1: +12V -> +24V
- R9 pad 2: GND -> +5V
- U1 pad 8: GND -> +5V
- U2 pad 4: GND -> +5V
- U2 pad 8: +12V -> +24V
Routing:
- net GND: track 11.8 -> 0.00 mm, vias 3 -> 0
- net +5V: track 0.00 -> 11.8 mm, vias 0 -> 3
- removed copper zone on B.Cu, net GND
- removed copper zone on F.Cu, net GND
Other:
- board text removed: "HIGH VOLTAGE!"
