File: IMD_Carrier/IMD_Carrier.kicad_sch (KiCad schematic)
At the start: 34 parts, among them IC1 CD4012BM96, J1 JST-XA, J2 MicroFit+, J3 JST-XA, J4 JST-XA, J5 JST-XA, K2 Relay_SPDT_G6RN, Q1 BSS205N, Q2 BSS205N, Q6 BSS205N, U1 CD4043BE, U2 TLV1702

Commit message: Add files via upload
Parts:
- removed IC1: CD4012BM96, Custom_MSM:Dual NAND, Quad input, symbol CD4012BM96:CD4012BM96
- added C10, C7: 10u, symbol Device:C
- added C11, C8: 100n, symbol Device:C
- added C3, C4: 0.1u, symbol Device:C
- added C5: 220u, symbol Device:C
- added C6: 680u, symbol Device:C
- added C9: 0.33u, symbol Device:C
- added D2, D5: D_TVS, symbol Device:D_TVS
- added D3: D_Schottky, symbol Device:D_Schottky
- added J6: MicroFit+, Custom_MSM:Connector_MicroFit-Plus_2POS, symbol Custom_MSM1:Connector_MicroFit-Plus_2POS
- added J7: JST-XA, Custom_MSM:Connector_JST-XA_4POS, symbol Custom_MSM1:Connector_JST-XA_4POS
- added L1: 33u, symbol Device:L
- added Q3: BSS205N, Custom_MSM:MOSFET_Single_SOT-23, symbol Custom_MSM:MOSFET_N-CH
- added Q4: BSS215P, Custom_MSM:MOSFET_Single_SOT-23, symbol Custom_MSM:MOSFET_P-CH
- added R12, R14: 10k, symbol Device:R
- added U3: LM2596S, Package_TO_SOT_SMD:TO-263-5_TabPin3, symbol Regulator_Switching:LM2596S-3.3
- added U4: BD450, Custom_MSM:Regulator_Linear_SOT-223-4, symbol Custom_MSM:Regulator_Linear_5V
- R10: value 8.5k -> 17k
- R11: value 3.5k -> 31k
- R8: value 2.5k -> 29k
- R9: value 9.5k -> 19k
Connections:
- net +12V: now also C10.1, C11.1, C5.1, C9.1, L1.2, U3.4 (FB), U4.1 (VI); no longer D4.1 (K), J1.2 (Pin_2), J4.1 (Pin_1), K2.5, R11.2, R13.1, R8.1, U2.8 (V+)
- net Chassis_GND: now also J7.3 (Pin_3)
- net HV+: now also J2.2 (Pin_2)
- net HV-: now also J6.1 (Pin_1), J6.2 (Pin_2); no longer J2.2 (Pin_2)
- net High_side_insulation: now also J7.1 (Pin_1)
- net IMD_Latch: now also Q3.1 (G)
- net IMD_fault: now also D5.2 (A2)
- net Low_side_insulation: now also J7.2 (Pin_2)
- net N_IMD_Latch: now also Q3.3 (D), R12.2
- net TSAC_GND: now also J7.4 (Pin_4)
- net GND renamed +5V
- net +5V: now also R13.1, C10.2, C11.2, C3.2, C4.2, C5.2, C6.2, C7.2, C8.1, C9.2, D2.1 (A1), D3.2 (A), D5.1 (A1), Q3.2 (S), R14.2, U3.3 (GND), U3.5 (~{ON}/OFF), U4.4 (GND)
- new net: J4.1 (Pin_1), Q4.3 (D)
- new net: D3.1 (K), L1.1, U3.2 (OUT)
- new net: C8.2, U4.2 (CTL)
- new net: C7.1, U4.3 (VO)
- new net: Q4.1 (G), R14.1
- new net +24V: C3.1, C4.1, C6.1, D2.2 (A2), D4.1 (K), J1.2 (Pin_2), K2.5, Q4.2 (S), R11.2, R12.1, R8.1, U2.8 (V+), U3.1 (VIN)
- no-connect marks 18 -> 11
Other:
- note added: "12-5V Regulator"
- note added: "24-12V Regulator"
- note added: "HV"
- note added: "LV"
- note added: "Voltage supression"
- moved on the sheet: J1, J2, J3, J4, J5, R10, R11, R13, R8, R9, TP1, TP2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
