File: IMD_Carrier-main/IMD_Carrier/IMD_Carrier.kicad_pcb (KiCad board)
At the start: 2 copper layers, 158 x 118 mm, 38 parts, among them IC1 CD4012BM96, J1 JST-XA, J2 MicroFit+, J3 JST-XA, J4 JST-XA, K2 Relay_SPDT_G6RN, Q1 BSS205N, Q2 BSS205N, Q6 BSS205N, U1 CD4043BE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

Commit message: FInished routing
Parts:
- D1: moved to F.Cu
- moved D1 3.41 mm to (120.6, 33.6), turned to 0 degrees
Routing:
- net Net-(D1-K): track 46.9 -> 81.9 mm, vias 1 -> 0
- net +12V: track 409.5 -> 396.9 mm, vias 4 -> 5
