File: IMD-Carrier/IMD-Carrier.kicad_pcb (KiCad board)
At the start: 2 copper layers, 158 x 118 mm, 65 parts, among them IC1 24-12V_Buck_reg, J1 JST-XA, J11 MicroFit+, J12 MicroFit+, J13 MicroFit+, J14 MicroFit+, J3 JST-XA, J4 JST-XA, J5 JST-XA, J7 JST-XA, K2 Relay_SPDT_G6RN, Q1 BSS205N, Q2 BSS205N, Q3 BSS205N, Q6 BSS205N, U1 CD4043BE, U2 TLV1702, U5 BD450

Commit message: Add files via upload
Parts:
- added G***: LOGO, LOGO, F.Cu at (168.4, 48.9)
- added G***: LOGO, Custom_MSM:Decorative_Stinger, F.Cu at (167.3, 130.1)
- added G***: LOGO, Custom_MSM:Decorative_TS_Hazard, F.Cu at (194.6, 41.2)
